Commit message: Use xacro to create a parameterized version of the car.

File: aav_car_ws/src/aav_simple_description/urdf/car.xacro (robot description, xacro)
@@ -1,92 +1,131 @@
 <?xml version="1.0"?>
 <robot name="car" xmlns:xacro="http://ros.org/wiki/xacro">
-    <link name="base_link">
-        <visual>
-            <origin xyz="0 0 0.3" rpy="0 0 0"/>
-            <geometry>
-                <box size="2.0 1.0 0.2"/>
-            </geometry>
-            <material name="green">
-                <color rgba="0 1 0 1"/>
-            </material>
-        </visual>
-    </link>
-    <link name="front_left_wheel">
-        <visual>
-            <origin xyz="0 0 0" rpy="0 1.5707 1.5707"/>
-            <geometry>
-                <cylinder radius="0.3" length="0.1"/>
-            </geometry>
-            <material name="black">
-                <color rbga="0 0 0 1"/>
-            </material>
-        </visual>
-    </link>
-    <link name="front_left_link"/>
-    <link name="front_right_wheel">
-        <visual>
-            <origin xyz="0 0 0" rpy="0 1.5707 1.5707"/>
-            <geometry>
-                <cylinder radius="0.3" length="0.1"/>
-            </geometry>
-            <material name="black"/>
-        </visual>
-    </link>
-    <link name="front_right_link"/>
-    <link name="back_left_wheel">
-        <visual>
-            <origin xyz="0 0 0" rpy="0 1.5707 1.5707"/>
-            <geometry>
-                <cylinder radius="0.3" length="0.1"/>
-            </geometry>
-            <material name="black"/>
-        </visual>
-    </link>
-    <link name="back_right_wheel">
-        <visual>
-            <origin xyz="0 0 0" rpy="0 1.5707 1.5707"/>
-            <geometry>
-                <cylinder radius="0.3" length="0.1"/>
-            </geometry>
-            <material name="black"/>
-        </visual>
-    </link>
-    <joint name="front_left_turn_joint" type="revolute">
-        <parent link="base_link"/>
-        <child link="front_left_link"/>
-        <origin xyz=".8 .6 .3"/>
-        <axis xyz="0 0 1"/>
-        <limit effort="1000" lower="-.548" upper=".548" velocity=".5"/>
-    </joint>
-    <joint name="front_left_joint" type="continuous">
-        <parent link="front_left_link"/>
-        <child link="front_left_wheel"/>
-        <axis xyz="0 1 0"/>
-    </joint>
-    <joint name="front_right_turn_joint" type="revolute">
-        <parent link="base_link"/>
-        <child link="front_right_link"/>
-        <origin xyz=".8 -.6 .3"/>
-        <axis xyz="0 0 1"/>
-        <limit effort="1000" lower="-.548" upper=".548" velocity=".5"/>
-        <mimic joint="front_left_turn_joint"/>
-    </joint>
-    <joint name="front_right_joint" type="continuous">
-        <parent link="front_right_link"/>
-        <child link="front_right_wheel"/>
-        <axis xyz="0 1 0"/>
-    </joint>
-    <joint name="back_left_joint" type="continuous">
-        <parent link="base_link"/>
-        <child link="back_left_wheel"/>
-        <axis xyz="0 1 0"/>
-        <origin xyz="-.8 .6 .3"/>
-    </joint>
-    <joint name="back_right_joint" type="continuous">
-        <parent link="base_link"/>
-        <child link="back_right_wheel"/>
-        <axis xyz="0 1 0"/>
-        <origin xyz="-.8 -.6 .3"/>
-        <mimic joint="back_left_joint"/>
-    </joint>
+  <!-- Axes are X (forward), Y (left), and Z (up).  This complies with the
+       right-hand rule.  Lengths are measured in meters and masses in
+       kilograms. -->
+  <!-- The dimensions of the car body itself. -->
+  <xacro:property name="chassis_length" value=".5334"/>
+  <xacro:property name="chassis_width" value=".28575"/>
+  <xacro:property name="chassis_height" value=".1397"/>
+  <!-- The distance between the ground to the bottom of the chassis. -->
+  <xacro:property name="ground_clearance" value=".05715"/>
+  <!-- -->
+  <xacro:property name="chassis_offset" value=".0254"/>
+  <!-- The center-to-center distance between the front wheels.  (It is assumed
+       that this is the same as the distance between the back wheels.) -->
+  <xacro:property name="wheelbase_width" value=".2413"/>
+  <!-- The distance between the front and back axes. -->
+  <xacro:property name="wheelbase_length" value=".3302"/>
+  <!-- The distance from the center of a wheel to the outside of its tire. -->
+  <xacro:property name="tire_radius" value=".0508"/>
+  <!-- The distance from the inside to the outside of a tire.  Basically, the
+       width of the tread. -->
+  <xacro:property name="tire_width" value=".047625"/>
+  <link name="base_link">
+    <visual>
+      <origin xyz="0 0 ${ground_clearance + chassis_height / 2}"/>
+      <geometry>
+        <box size="${chassis_length} ${chassis_width} ${chassis_height}"/>
+      </geometry>
+      <material name="blue">
+        <color rgba="0 0 1 1"/>
+      </material>
+    </visual>
+  </link>
+  <link name="front_left_wheel">
+    <visual>
+      <origin xyz="0 0 0" rpy="0 1.5707 1.5707"/>
+      <geometry>
+        <cylinder radius="${tire_radius}" length="${tire_width}"/>
+      </geometry>
+      <material name="black">
+        <color rgba="0 0 0 1"/>
+      </material>
+    </visual>
+  </link>
+  <link name="front_left_link"/>
+  <joint name="front_left_turn_joint" type="revolute">
+    <parent link="base_link"/>
+    <child link="front_left_link"/>
+    <origin xyz="${wheelbase_length / 2} -${wheelbase_width / 2} ${tire_radius}"/>
+    <axis xyz="0 0 1"/>
+    <limit effort="1000" lower="-.548" upper=".548" velocity=".5"/>
+  </joint>
+  <joint name="front_left_joint" type="continuous">
+    <parent link="front_left_link"/>
+    <child link="front_left_wheel"/>
+    <axis xyz="0 1 0"/>
+  </joint>
+  <link name="front_right_wheel">
+    <visual>
+      <origin xyz="0 0 0" rpy="0 1.5707 1.5707"/>
+      <geometry>
+        <cylinder radius="${tire_radius}" length="${tire_width}"/>
+      </geometry>
+      <material name="black">
+        <color rgba="0 0 0 1"/>
+      </material>
+    </visual>
+  </link>
+  <link name="front_right_link"/>
+  <joint name="front_right_turn_joint" type="revolute">
+    <parent link="base_link"/>
+    <child link="front_right_link"/>
+    <origin xyz="${wheelbase_length / 2} ${wheelbase_width / 2} ${tire_radius}"/>
+    <axis xyz="0 0 1"/>
+    <limit effort="1000" lower="-.548" upper=".548" velocity=".5"/>
+  </joint>
+  <joint name="front_right_joint" type="continuous">
+    <parent link="front_right_link"/>
+    <child link="front_right_wheel"/>
+    <axis xyz="0 1 0"/>
+  </joint>
+  <link name="rear_left_wheel">
+    <visual>
+      <origin xyz="0 0 0" rpy="0 1.5707 1.5707"/>
+      <geometry>
+        <cylinder radius="${tire_radius}" length="${tire_width}"/>
+      </geometry>
+      <material name="black">
+        <color rgba="0 0 0 1"/>
+      </material>
+    </visual>
+  </link>
+  <link name="rear_left_link"/>
+  <joint name="rear_left_turn_joint" type="revolute">
+    <parent link="base_link"/>
+    <child link="rear_left_link"/>
+    <origin xyz="-${wheelbase_length / 2} -${wheelbase_width / 2} ${tire_radius}"/>
+    <axis xyz="0 0 1"/>
+    <limit effort="1000" lower="-.548" upper=".548" velocity=".5"/>
+  </joint>
+  <joint name="rear_left_joint" type="continuous">
+    <parent link="rear_left_link"/>
+    <child link="rear_left_wheel"/>
+    <axis xyz="0 1 0"/>
+  </joint>
+  <link name="rear_right_wheel">
+    <visual>
+      <origin xyz="0 0 0" rpy="0 1.5707 1.5707"/>
+      <geometry>
+        <cylinder radius="${tire_radius}" length="${tire_width}"/>
+      </geometry>
+      <material name="black">
+        <color rgba="0 0 0 1"/>
+      </material>
+    </visual>
+  </link>
+  <link name="rear_right_link"/>
+  <joint name="rear_right_turn_joint" type="revolute">
+    <parent link="base_link"/>
+    <child link="rear_right_link"/>
+    <origin xyz="-${wheelbase_length / 2} ${wheelbase_width / 2} ${tire_radius}"/>
+    <axis xyz="0 0 1"/>
+    <limit effort="1000" lower="-.548" upper=".548" velocity=".5"/>
+  </joint>
+  <joint name="rear_right_joint" type="continuous">
+    <parent link="rear_right_link"/>
+    <child link="rear_right_wheel"/>
+    <axis xyz="0 1 0"/>
+  </joint>
 </robot>

Commit message: Use xacro to reduce the duplication between each wheel.

File: aav_car_ws/src/aav_simple_description/urdf/car.xacro (robot description, xacro)
@@ -22,4 +22,53 @@
        width of the tread. -->
   <xacro:property name="tire_width" value=".047625"/>
+  <xacro:macro name="front_wheel" params="name x">
+    <link name="front_${name}_wheel">
+      <visual>
+        <origin xyz="0 0 0" rpy="0 1.5707 1.5707"/>
+        <geometry>
+          <cylinder radius="${tire_radius}" length="${tire_width}"/>
+        </geometry>
+        <material name="black">
+          <color rgba="0 0 0 1"/>
+        </material>
+      </visual>
+    </link>
+    <link name="front_${name}_link"/>
+    <joint name="front_${name}_turn_joint" type="revolute">
+      <parent link="base_link"/>
+      <child link="front_${name}_link"/>
+      <origin xyz="${wheelbase_length / 2}
+        ${x * wheelbase_width / 2}
+        ${tire_radius}"/>
+      <axis xyz="0 0 1"/>
+      <limit effort="1000" lower="-.548" upper=".548" velocity=".5"/>
+    </joint>
+    <joint name="front_${name}_joint" type="continuous">
+      <parent link="front_${name}_link"/>
+      <child link="front_${name}_wheel"/>
+      <axis xyz="0 1 0"/>
+    </joint>
+  </xacro:macro>
+  <xacro:macro name="back_wheel" params="name x">
+    <link name="back_${name}_wheel">
+      <visual>
+        <origin xyz="0 0 0" rpy="0 1.5707 1.5707"/>
+        <geometry>
+          <cylinder radius="${tire_radius}" length="${tire_width}"/>
+        </geometry>
+        <material name="black">
+          <color rgba="0 0 0 1"/>
+        </material>
+      </visual>
+    </link>
+    <joint name="back_${name}_joint" type="continuous">
+      <parent link="base_link"/>
+      <child link="back_${name}_wheel"/>
+      <axis xyz="0 1 0"/>
+      <origin xyz="${-wheelbase_length / 2}
+        ${x * wheelbase_width / 2}
+        ${tire_radius}"/>
+    </joint>
+  </xacro:macro>
   <link name="base_link">
     <visual>
@@ -33,99 +82,7 @@
     </visual>
   </link>
-  <link name="front_left_wheel">
-    <visual>
-      <origin xyz="0 0 0" rpy="0 1.5707 1.5707"/>
-      <geometry>
-        <cylinder radius="${tire_radius}" length="${tire_width}"/>
-      </geometry>
-      <material name="black">
-        <color rgba="0 0 0 1"/>
-      </material>
-    </visual>
-  </link>
-  <link name="front_left_link"/>
-  <joint name="front_left_turn_joint" type="revolute">
-    <parent link="base_link"/>
-    <child link="front_left_link"/>
-    <origin xyz="${wheelbase_length / 2} -${wheelbase_width / 2} ${tire_radius}"/>
-    <axis xyz="0 0 1"/>
-    <limit effort="1000" lower="-.548" upper=".548" velocity=".5"/>
-  </joint>
-  <joint name="front_left_joint" type="continuous">
-    <parent link="front_left_link"/>
-    <child link="front_left_wheel"/>
-    <axis xyz="0 1 0"/>
-  </joint>
-  <link name="front_right_wheel">
-    <visual>
-      <origin xyz="0 0 0" rpy="0 1.5707 1.5707"/>
-      <geometry>
-        <cylinder radius="${tire_radius}" length="${tire_width}"/>
-      </geometry>
-      <material name="black">
-        <color rgba="0 0 0 1"/>
-      </material>
-    </visual>
-  </link>
-  <link name="front_right_link"/>
-  <joint name="front_right_turn_joint" type="revolute">
-    <parent link="base_link"/>
-    <child link="front_right_link"/>
-    <origin xyz="${wheelbase_length / 2} ${wheelbase_width / 2} ${tire_radius}"/>
-    <axis xyz="0 0 1"/>
-    <limit effort="1000" lower="-.548" upper=".548" velocity=".5"/>
-  </joint>
-  <joint name="front_right_joint" type="continuous">
-    <parent link="front_right_link"/>
-    <child link="front_right_wheel"/>
-    <axis xyz="0 1 0"/>
-  </joint>
-  <link name="rear_left_wheel">
-    <visual>
-      <origin xyz="0 0 0" rpy="0 1.5707 1.5707"/>
-      <geometry>
-        <cylinder radius="${tire_radius}" length="${tire_width}"/>
-      </geometry>
-      <material name="black">
-        <color rgba="0 0 0 1"/>
-      </material>
-    </visual>
-  </link>
-  <link name="rear_left_link"/>
-  <joint name="rear_left_turn_joint" type="revolute">
-    <parent link="base_link"/>
-    <child link="rear_left_link"/>
-    <origin xyz="-${wheelbase_length / 2} -${wheelbase_width / 2} ${tire_radius}"/>
-    <axis xyz="0 0 1"/>
-    <limit effort="1000" lower="-.548" upper=".548" velocity=".5"/>
-  </joint>
-  <joint name="rear_left_joint" type="continuous">
-    <parent link="rear_left_link"/>
-    <child link="rear_left_wheel"/>
-    <axis xyz="0 1 0"/>
-  </joint>
-  <link name="rear_right_wheel">
-    <visual>
-      <origin xyz="0 0 0" rpy="0 1.5707 1.5707"/>
-      <geometry>
-        <cylinder radius="${tire_radius}" length="${tire_width}"/>
-      </geometry>
-      <material name="black">
-        <color rgba="0 0 0 1"/>
-      </material>
-    </visual>
-  </link>
-  <link name="rear_right_link"/>
-  <joint name="rear_right_turn_joint" type="revolute">
-    <parent link="base_link"/>
-    <child link="rear_right_link"/>
-    <origin xyz="-${wheelbase_length / 2} ${wheelbase_width / 2} ${tire_radius}"/>
-    <axis xyz="0 0 1"/>
-    <limit effort="1000" lower="-.548" upper=".548" velocity=".5"/>
-  </joint>
-  <joint name="rear_right_joint" type="continuous">
-    <parent link="rear_right_link"/>
-    <child link="rear_right_wheel"/>
-    <axis xyz="0 1 0"/>
-  </joint>
+  <xacro:front_wheel name="left" x="-1"/>
+  <xacro:front_wheel name="right" x="1"/>
+  <xacro:back_wheel name="left" x="-1"/>
+  <xacro:back_wheel name="right" x="1"/>
 </robot>
