Commit message: Begin modifying the URDF file to work in Gazebo.

File: aav_car_ws/src/aav_simple_description/urdf/car.urdf.xacro (robot description, xacro)
@@ -7,4 +7,10 @@
   <xacro:include filename="$(find aav_simple_description)/urdf/wheel.urdf.xacro"/>
   <link name="base_link">
+    <collision>
+      <origin xyz="0 0 ${ground_clearance + chassis_height / 2}"/>
+      <geometry>
+        <box size="${chassis_length} ${chassis_width} ${chassis_height}"/>
+      </geometry>
+    </collision>
     <visual>
       <origin xyz="0 0 ${ground_clearance + chassis_height / 2}"/>
@@ -16,5 +22,14 @@
       </material>
     </visual>
+    <inertial>
+      <origin xyz="0 0 ${ground_clearance + chassis_height / 2}"/>
+      <mass value="2.26796"/>
+      <inertia ixx="1" ixy="0" ixz="0" iyy="1" iyz="0" izz="1"/>
+    </inertial>
   </link>
+  <gazebo reference="base_link">
+    <material>Gazebo/Blue</material>
+    <turnGravityOff>false</turnGravityOff>
+  </gazebo>
   <xacro:front_wheel name="left" x="-1"/>
   <xacro:front_wheel name="right" x="1"/>

File: aav_car_ws/src/aav_simple_description/urdf/wheel.urdf.xacro (robot description, xacro)
@@ -3,4 +3,10 @@
   <xacro:macro name="front_wheel" params="name x">
     <link name="front_${name}_wheel">
+      <collision>
+        <origin xyz="0 0 0" rpy="0 1.5707 1.5707"/>
+        <geometry>
+          <cylinder radius="${tire_radius}" length="${tire_width}"/>
+        </geometry>
+      </collision>
       <visual>
         <origin xyz="0 0 0" rpy="0 1.5707 1.5707"/>
@@ -12,6 +18,21 @@
         </material>
       </visual>
+      <inertial>
+        <origin xyz="0 0 0" rpy="0 1.5707 1.5707"/>
+        <mass value=".5"/>
+        <inertia ixx="1" ixy="0" ixz="0" iyy="1" iyz="0" izz="1"/>
+      </inertial>
     </link>
-    <link name="front_${name}_link"/>
+    <gazebo reference="front_${name}_wheel">
+      <material>Gazebo/Black</material>
+      <turnGravityOff>false</turnGravityOff>
+    </gazebo>
+    <link name="front_${name}_link">
+      <inertial>
+        <origin xyz="0 0 0"/>
+        <mass value="1"/>
+        <inertia ixx="1" ixy="0" ixz="0" iyy="1" iyz="0" izz="1"/>
+      </inertial>
+    </link>
     <joint name="front_${name}_turn_joint" type="revolute">
       <parent link="base_link"/>
@@ -26,4 +47,5 @@
       <parent link="front_${name}_link"/>
       <child link="front_${name}_wheel"/>
+      <origin xyz="0 0 0"/>
       <axis xyz="0 1 0"/>
     </joint>
@@ -31,4 +53,10 @@
   <xacro:macro name="back_wheel" params="name x">
     <link name="back_${name}_wheel">
+      <collision>
+        <origin xyz="0 0 0" rpy="0 1.5707 1.5707"/>
+        <geometry>
+          <cylinder radius="${tire_radius}" length="${tire_width}"/>
+        </geometry>
+      </collision>
       <visual>
         <origin xyz="0 0 0" rpy="0 1.5707 1.5707"/>
@@ -40,5 +68,13 @@
         </material>
       </visual>
+      <inertial>
+        <origin xyz="0 0 0" rpy="0 1.5707 1.5707"/>
+        <mass value=".5"/>
+        <inertia ixx="1" ixy="0" ixz="0" iyy="1" iyz="0" izz="1"/>
+      </inertial>
     </link>
+    <gazebo reference="back_${name}_wheel">
+      <material>Gazebo/Black</material>
+    </gazebo>
     <joint name="back_${name}_joint" type="continuous">
       <parent link="base_link"/>

Commit message: Get the wheels turning.

File: aav_car_ws/src/aav_simple_description/urdf/car.urdf.xacro (robot description, xacro)
@@ -28,5 +28,6 @@
       <origin xyz="0 0 ${ground_clearance + chassis_height / 2}"/>
       <mass value="2.26796"/>
-      <inertia ixx="1" ixy="0" ixz="0" iyy="1" iyz="0" izz="1"/>
+      <inertia ixx=".0065806093" ixy="0" ixz="0"
+        iyy=".0154882693" iyz="0" izz=".0220224112"/>
     </inertial>
   </link>

File: aav_car_ws/src/aav_simple_description/urdf/wheel.urdf.xacro (robot description, xacro)
@@ -21,5 +21,5 @@
         <origin xyz="0 0 0" rpy="0 1.5707 1.5707"/>
         <mass value=".5"/>
-        <inertia ixx="1" ixy="0" ixz="0" iyy="1" iyz="0" izz="1"/>
+        <inertia ixx=".02467" ixy="0" ixz="0" iyy=".02467" iyz="0" izz=".04411"/>
       </inertial>
     </link>
@@ -27,10 +27,15 @@
       <material>Gazebo/Black</material>
       <turnGravityOff>false</turnGravityOff>
+      <mu1 value="1"/>
+      <mu2 value="1"/>
+      <kp value="10000000"/>
+      <kd value="1"/>
+      <fdir1 value="1 0 0"/>
     </gazebo>
     <link name="front_${name}_link">
       <inertial>
         <origin xyz="0 0 0"/>
-        <mass value="1"/>
-        <inertia ixx="1" ixy="0" ixz="0" iyy="1" iyz="0" izz="1"/>
+        <mass value=".6"/>
+        <inertia ixx=".001" ixy="0" ixz="0" iyy=".001" iyz="0" izz=".001"/>
       </inertial>
     </link>
@@ -71,9 +76,15 @@
         <origin xyz="0 0 0" rpy="0 1.5707 1.5707"/>
         <mass value=".5"/>
-        <inertia ixx="1" ixy="0" ixz="0" iyy="1" iyz="0" izz="1"/>
+        <inertia ixx=".02467" ixy="0" ixz="0" iyy=".02467" iyz="0" izz=".04411"/>
       </inertial>
     </link>
     <gazebo reference="back_${name}_wheel">
       <material>Gazebo/Black</material>
+      <turnGravityOff>false</turnGravityOff>
+      <mu1 value="1.5"/>
+      <mu2 value="1.5"/>
+      <kp value="1000000"/>
+      <kd value="100"/>
+      <fdir1 value="1 0 0"/>
     </gazebo>
     <joint name="back_${name}_joint" type="continuous">
