Commit message: Create an aav_control package.

File: aav_car_ws/src/aav_description/urdf/car.urdf.xacro (robot description, xacro)
@@ -359,3 +359,37 @@
     <plugin name="gazebo_ros_control" filename="libgazebo_ros_control.so"/>
   </gazebo>
+  <link name="imu_link"/>
+  <joint name="imu_joint" type="fixed">
+    <parent link="chassis"/>
+    <child link="imu_link"/>
+  </joint>
+  <gazebo>
+    <plugin name="imu_controller" filename="libhector_gazebo_ros_imu.so">
+      <robotNamespace>/</robotNamespace>
+      <updateRate>50.0</updateRate>
+      <bodyName>base_link</bodyName>
+      <topicName>imu/data_compass</topicName>
+      <accelDrift>0.005 0.005 0.005</accelDrift>
+      <accelGaussianNoise>0.005 0.005 0.005</accelGaussianNoise>
+      <rateDrift>0.005 0.005 0.005 </rateDrift>
+      <rateGaussianNoise>0.005 0.005 0.005 </rateGaussianNoise>
+      <headingDrift>0.005</headingDrift>
+      <headingGaussianNoise>0.005</headingGaussianNoise>
+    </plugin>
+  </gazebo>
+  <gazebo>
+    <plugin name="gps_controller" filename="libhector_gazebo_ros_gps.so">
+      <updateRate>10</updateRate>
+      <robotNamespace>/</robotNamespace>
+      <bodyName>base_link</bodyName>
+      <frameId>base_link</frameId>
+      <topicName>navsat/fix</topicName>
+      <velocityTopicName>navsat/vel</velocityTopicName>
+      <referenceLatitude>43.547165</referenceLatitude>
+      <referenceLongitude>-116.330745</referenceLongitude>
+      <referenceHeading>0</referenceHeading>
+      <referenceAltitude>824</referenceAltitude>
+      <drift>0.0001 0.0001 0.0001</drift>
+    </plugin>
+  </gazebo>
 </robot>

Commit message: Add a link to be used for calculating the CTE.

File: aav_car_ws/src/aav_description/urdf/car.urdf.xacro (robot description, xacro)
@@ -316,4 +316,17 @@
     <material>Gazebo/Grey</material>
   </gazebo>
+  <link name="unicycle_pivot">
+    <visual>
+      <geometry>
+        <box size="0.01 0.01 0.01"/>
+      </geometry>
+      <material name="chassis_mat"/>
+    </visual>
+  </link>
+  <joint name="base_link_to_unicycle_pivot" type="fixed">
+    <parent link="base_link"/>
+    <child link="unicycle_pivot"/>
+    <origin xyz="${wheelbase / 2} 0 0"/>
+  </joint>
   <!-- Chassis -->
   <link name="chassis">

Commit message: Just reposition the base_link instead of creating a new link to calculate the CTE.

File: aav_car_ws/src/aav_description/urdf/car.urdf.xacro (robot description, xacro)
@@ -316,17 +316,4 @@
     <material>Gazebo/Grey</material>
   </gazebo>
-  <link name="unicycle_pivot">
-    <visual>
-      <geometry>
-        <box size="0.01 0.01 0.01"/>
-      </geometry>
-      <material name="chassis_mat"/>
-    </visual>
-  </link>
-  <joint name="base_link_to_unicycle_pivot" type="fixed">
-    <parent link="base_link"/>
-    <child link="unicycle_pivot"/>
-    <origin xyz="${wheelbase / 2} 0 0"/>
-  </joint>
   <!-- Chassis -->
   <link name="chassis">
@@ -353,7 +340,8 @@
     <material>Gazebo/Grey</material>
   </gazebo>
-  <joint name="base_link_to_chasis" type="fixed">
+  <joint name="base_link_to_chassis" type="fixed">
     <parent link="base_link"/>
     <child link="chassis"/>
+    <origin xyz="-${wheelbase / 2} 0 0"/>
   </joint>
   <!-- Batteries -->
